File: ferris.sch (KiCad schematic (older format))
At the start: 95 parts, among them J1 USB C, K0_0 KEYSW, K0_1 KEYSW, K0_2 KEYSW, K0_3 KEYSW, K0_4 KEYSW, K0_5 KEYSW, K0_6 KEYSW, K0_7 KEYSW, K0_8 KEYSW, K0_9 KEYSW, K1_0 KEYSW, K1_1 KEYSW, K1_2 KEYSW, K1_3 KEYSW, K1_4 KEYSW, K1_5 KEYSW, K1_6 KEYSW, K1_7 KEYSW, K1_8 KEYSW, K1_9 KEYSW, K2_0 KEYSW, K2_1 KEYSW, K2_2 KEYSW, K2_3 KEYSW, K2_4 KEYSW, K2_5 KEYSW, K2_6 KEYSW, K2_7 KEYSW, K2_8 KEYSW, K2_9 KEYSW, K3_3 KEYSW, K3_4 KEYSW, K3_5 KEYSW, K3_6 KEYSW, SW1 SW_PUSH, U1 ATmega32U4-AU, U2 MCP23017_SO, Y1 Crystal

Commit message: Design the "Ferris low" variant
* Same as the base variant with major change that the footprints are
  for Kailh PG1232 instead of choc for an even lower profile
* Copper pad adapted to ducking Ferris for theme
* Silkscreen changed to display schematics from the PG1232 switch
* Recommended PCB solder mask color is blue instead of white so the
  silkscreen gives vibes of a blueprint
* Name of the board updated to "Ferris low" instead of "Ferris"
Parts:
- K0_0, K0_1, K0_2, K0_3, K0_4, K0_5, K0_6, K0_7, K0_8, K0_9, K1_0, K1_1, K1_2, K1_3, K1_4, K1_5, K1_6, K1_7, K1_8, K1_9, K2_0, K2_1, K2_2, K2_3, K2_4, K2_5, K2_6, K2_7, K2_8, K2_9, K3_3, K3_4, K3_5, K3_6: footprint ferris:SW_PG1350 -> ferris:Kailh_PG1232
Changed lines of the file:
@@
 F 0 "K0_0" H 1350 1433 60  0000 C CNN
 F 1 "KEYSW" H 1350 1100 60  0001 C CNN
-F 2 "ferris:SW_PG1350" H 1350 1200 60  0001 C CNN
+F 2 "ferris:Kailh_PG1232" H 1350 1200 60  0001 C CNN
 F 3 "" H 1350 1200 60  0000 C CNN
 F 4 "C489144" H 1350 1200 50  0001 C CNN "LCSC Part #"
@@
 F 0 "K1_0" H 1350 2033 60  0000 C CNN
 F 1 "KEYSW" H 1350 1700 60  0001 C CNN
-F 2 "ferris:SW_PG1350" H 1350 1800 60  0001 C CNN
+F 2 "ferris:Kailh_PG1232" H 1350 1800 60  0001 C CNN
 F 3 "" H 1350 1800 60  0000 C CNN
 	1    1350 1800
@@
 F 0 "K1_1" H 2050 2033 60  0000 C CNN
 F 1 "KEYSW" H 2050 1700 60  0001 C CNN
-F 2 "ferris:SW_PG1350" H 2050 1800 60  0001 C CNN
+F 2 "ferris:Kailh_PG1232" H 2050 1800 60  0001 C CNN
 F 3 "" H 2050 1800 60  0000 C CNN
 	1    2050 1800
@@
 F 0 "K0_2" H 2750 1433 60  0000 C CNN
 F 1 "KEYSW" H 2750 1100 60  0001 C CNN
-F 2 "ferris:SW_PG1350" H 2750 1200 60  0001 C CNN
+F 2 "ferris:Kailh_PG1232" H 2750 1200 60  0001 C CNN
 F 3 "" H 2750 1200 60  0000 C CNN
 	1    2750 1200
@@
 F 0 "K0_1" H 2050 1433 60  0000 C CNN
 F 1 "KEYSW" H 2050 1100 60  0001 C CNN
-F 2 "ferris:SW_PG1350" H 2050 1200 60  0001 C CNN
+F 2 "ferris:Kailh_PG1232" H 2050 1200 60  0001 C CNN
 F 3 "" H 2050 1200 60  0000 C CNN
 	1    2050 1200
@@
 F 0 "K1_2" H 2750 2033 60  0000 C CNN
 F 1 "KEYSW" H 2750 1700 60  0001 C CNN
-F 2 "ferris:SW_PG1350" H 2750 1800 60  0001 C CNN
+F 2 "ferris:Kailh_PG1232" H 2750 1800 60  0001 C CNN
 F 3 "" H 2750 1800 60  0000 C CNN
 	1    2750 1800
@@
 F 0 "K2_0" H 1350 2633 60  0000 C CNN
 F 1 "KEYSW" H 1350 2300 60  0001 C CNN
-F 2 "ferris:SW_PG1350" H 1350 2400 60  0001 C CNN
+F 2 "ferris:Kailh_PG1232" H 1350 2400 60  0001 C CNN
 F 3 "" H 1350 2400 60  0000 C CNN
 	1    1350 2400
@@
 F 0 "K2_1" H 2050 2633 60  0000 C CNN
 F 1 "KEYSW" H 2050 2300 60  0001 C CNN
-F 2 "ferris:SW_PG1350" H 2050 2400 60  0001 C CNN
+F 2 "ferris:Kailh_PG1232" H 2050 2400 60  0001 C CNN
 F 3 "" H 2050 2400 60  0000 C CNN
 	1    2050 2400
@@
 F 0 "K2_2" H 2750 2633 60  0000 C CNN
 F 1 "KEYSW" H 2750 2300 60  0001 C CNN
-F 2 "ferris:SW_PG1350" H 2750 2400 60  0001 C CNN
+F 2 "ferris:Kailh_PG1232" H 2750 2400 60  0001 C CNN
 F 3 "" H 2750 2400 60  0000 C CNN
 	1    2750 2400
@@
 F 0 "K0_3" H 3450 1433 60  0000 C CNN
 F 1 "KEYSW" H 3450 1100 60  0001 C CNN
-F 2 "ferris:SW_PG1350" H 3450 1200 60  0001 C CNN
+F 2 "ferris:Kailh_PG1232" H 3450 1200 60  0001 C CNN
 F 3 "" H 3450 1200 60  0000 C CNN
 	1    3450 1200
@@
 F 0 "K1_3" H 3450 2033 60  0000 C CNN
 F 1 "KEYSW" H 3450 1700 60  0001 C CNN
-F 2 "ferris:SW_PG1350" H 3450 1800 60  0001 C CNN
+F 2 "ferris:Kailh_PG1232" H 3450 1800 60  0001 C CNN
 F 3 "" H 3450 1800 60  0000 C CNN
 	1    3450 1800
@@
 F 0 "K2_3" H 3450 2633 60  0000 C CNN
 F 1 "KEYSW" H 3450 2300 60  0001 C CNN
-F 2 "ferris:SW_PG1350" H 3450 2400 60  0001 C CNN
+F 2 "ferris:Kailh_PG1232" H 3450 2400 60  0001 C CNN
 F 3 "" H 3450 2400 60  0000 C CNN
 	1    3450 2400
@@
 F 0 "K0_4" H 4150 1433 60  0000 C CNN
 F 1 "KEYSW" H 4150 1100 60  0001 C CNN
-F 2 "ferris:SW_PG1350" H 4150 1200 60  0001 C CNN
+F 2 "ferris:Kailh_PG1232" H 4150 1200 60  0001 C CNN
 F 3 "" H 4150 1200 60  0000 C CNN
 	1    4150 1200
@@
 F 0 "K1_4" H 4150 2033 60  0000 C CNN
 F 1 "KEYSW" H 4150 1700 60  0001 C CNN
-F 2 "ferris:SW_PG1350" H 4150 1800 60  0001 C CNN
+F 2 "ferris:Kailh_PG1232" H 4150 1800 60  0001 C CNN
 F 3 "" H 4150 1800 60  0000 C CNN
 	1    4150 1800
@@
 F 0 "K2_4" H 4150 2633 60  0000 C CNN
 F 1 "KEYSW" H 4150 2300 60  0001 C CNN
-F 2 "ferris:SW_PG1350" H 4150 2400 60  0001 C CNN
+F 2 "ferris:Kailh_PG1232" H 4150 2400 60  0001 C CNN
 F 3 "" H 4150 2400 60  0000 C CNN
 	1    4150 2400
@@
 F 0 "K3_3" H 3450 3233 60  0000 C CNN
 F 1 "KEYSW" H 3450 2900 60  0001 C CNN
-F 2 "ferris:SW_PG1350" H 3450 3000 60  0001 C CNN
+F 2 "ferris:Kailh_PG1232" H 3450 3000 60  0001 C CNN
 F 3 "" H 3450 3000 60  0000 C CNN
 	1    3450 3000
@@
 F 0 "K3_4" H 4150 3233 60  0000 C CNN
 F 1 "KEYSW" H 4150 2900 60  0001 C CNN
-F 2 "ferris:SW_PG1350" H 4150 3000 60  0001 C CNN
+F 2 "ferris:Kailh_PG1232" H 4150 3000 60  0001 C CNN
 F 3 "" H 4150 3000 60  0000 C CNN
 	1    4150 3000
@@
 F 0 "K0_5" H 7450 1433 60  0000 C CNN
 F 1 "KEYSW" H 7450 1100 60  0001 C CNN
-F 2 "ferris:SW_PG1350" H 7450 1200 60  0001 C CNN
+F 2 "ferris:Kailh_PG1232" H 7450 1200 60  0001 C CNN
 F 3 "" H 7450 1200 60  0000 C CNN
 	1    7450 1200
@@
 F 0 "K1_5" H 7450 2033 60  0000 C CNN
 F 1 "KEYSW" H 7450 1700 60  0001 C CNN
-F 2 "ferris:SW_PG1350" H 7450 1800 60  0001 C CNN
+F 2 "ferris:Kailh_PG1232" H 7450 1800 60  0001 C CNN
 F 3 "" H 7450 1800 60  0000 C CNN
 	1    7450 1800
@@
 F 0 "K1_6" H 8150 2033 60  0000 C CNN
 F 1 "KEYSW" H 8150 1700 60  0001 C CNN
-F 2 "ferris:SW_PG1350" H 8150 1800 60  0001 C CNN
+F 2 "ferris:Kailh_PG1232" H 8150 1800 60  0001 C CNN
 F 3 "" H 8150 1800 60  0000 C CNN
 	1    8150 1800
@@
 F 0 "K0_7" H 8850 1433 60  0000 C CNN
 F 1 "KEYSW" H 8850 1100 60  0001 C CNN
-F 2 "ferris:SW_PG1350" H 8850 1200 60  0001 C CNN
+F 2 "ferris:Kailh_PG1232" H 8850 1200 60  0001 C CNN
 F 3 "" H 8850 1200 60  0000 C CNN
 	1    8850 1200
@@
 F 0 "K0_6" H 8150 1433 60  0000 C CNN
 F 1 "KEYSW" H 8150 1100 60  0001 C CNN
-F 2 "ferris:SW_PG1350" H 8150 1200 60  0001 C CNN
+F 2 "ferris:Kailh_PG1232" H 8150 1200 60  0001 C CNN
 F 3 "" H 8150 1200 60  0000 C CNN
 	1    8150 1200
@@
 F 0 "K1_7" H 8850 2033 60  0000 C CNN
 F 1 "KEYSW" H 8850 1700 60  0001 C CNN
-F 2 "ferris:SW_PG1350" H 8850 1800 60  0001 C CNN
+F 2 "ferris:Kailh_PG1232" H 8850 1800 60  0001 C CNN
 F 3 "" H 8850 1800 60  0000 C CNN
 	1    8850 1800
@@
 F 0 "K2_5" H 7450 2633 60  0000 C CNN
 F 1 "KEYSW" H 7450 2300 60  0001 C CNN
-F 2 "ferris:SW_PG1350" H 7450 2400 60  0001 C CNN
+F 2 "ferris:Kailh_PG1232" H 7450 2400 60  0001 C CNN
 F 3 "" H 7450 2400 60  0000 C CNN
 	1    7450 2400
@@
 F 0 "K2_6" H 8150 2633 60  0000 C CNN
 F 1 "KEYSW" H 8150 2300 60  0001 C CNN
-F 2 "ferris:SW_PG1350" H 8150 2400 60  0001 C CNN
+F 2 "ferris:Kailh_PG1232" H 8150 2400 60  0001 C CNN
 F 3 "" H 8150 2400 60  0000 C CNN
 	1    8150 2400
@@
 F 0 "K2_7" H 8850 2633 60  0000 C CNN
 F 1 "KEYSW" H 8850 2300 60  0001 C CNN
-F 2 "ferris:SW_PG1350" H 8850 2400 60  0001 C CNN
+F 2 "ferris:Kailh_PG1232" H 8850 2400 60  0001 C CNN
 F 3 "" H 8850 2400 60  0000 C CNN
 	1    8850 2400
@@
 F 0 "K0_8" H 9550 1433 60  0000 C CNN
 F 1 "KEYSW" H 9550 1100 60  0001 C CNN
-F 2 "ferris:SW_PG1350" H 9550 1200 60  0001 C CNN
+F 2 "ferris:Kailh_PG1232" H 9550 1200 60  0001 C CNN
 F 3 "" H 9550 1200 60  0000 C CNN
 	1    9550 1200
@@
 F 0 "K1_8" H 9550 2033 60  0000 C CNN
 F 1 "KEYSW" H 9550 1700 60  0001 C CNN
-F 2 "ferris:SW_PG1350" H 9550 1800 60  0001 C CNN
+F 2 "ferris:Kailh_PG1232" H 9550 1800 60  0001 C CNN
 F 3 "" H 9550 1800 60  0000 C CNN
 	1    9550 1800
@@
 F 0 "K2_8" H 9550 2633 60  0000 C CNN
 F 1 "KEYSW" H 9550 2300 60  0001 C CNN
-F 2 "ferris:SW_PG1350" H 9550 2400 60  0001 C CNN
+F 2 "ferris:Kailh_PG1232" H 9550 2400 60  0001 C CNN
 F 3 "" H 9550 2400 60  0000 C CNN
 	1    9550 2400
@@
 F 0 "K0_9" H 10250 1433 60  0000 C CNN
 F 1 "KEYSW" H 10250 1100 60  0001 C CNN
-F 2 "ferris:SW_PG1350" H 10250 1200 60  0001 C CNN
+F 2 "ferris:Kailh_PG1232" H 10250 1200 60  0001 C CNN
 F 3 "" H 10250 1200 60  0000 C CNN
 	1    10250 1200
@@
 F 0 "K1_9" H 10250 2033 60  0000 C CNN
 F 1 "KEYSW" H 10250 1700 60  0001 C CNN
-F 2 "ferris:SW_PG1350" H 10250 1800 60  0001 C CNN
+F 2 "ferris:Kailh_PG1232" H 10250 1800 60  0001 C CNN
 F 3 "" H 10250 1800 60  0000 C CNN
 	1    10250 1800
@@
 F 0 "K2_9" H 10250 2633 60  0000 C CNN
 F 1 "KEYSW" H 10250 2300 60  0001 C CNN
-F 2 "ferris:SW_PG1350" H 10250 2400 60  0001 C CNN
+F 2 "ferris:Kailh_PG1232" H 10250 2400 60  0001 C CNN
 F 3 "" H 10250 2400 60  0000 C CNN
 	1    10250 2400
@@
 F 0 "K3_5" H 7450 3233 60  0000 C CNN
 F 1 "KEYSW" H 7450 2900 60  0001 C CNN
-F 2 "ferris:SW_PG1350" H 7450 3000 60  0001 C CNN
+F 2 "ferris:Kailh_PG1232" H 7450 3000 60  0001 C CNN
 F 3 "" H 7450 3000 60  0000 C CNN
 	1    7450 3000
@@
 F 0 "K3_6" H 8150 3233 60  0000 C CNN
 F 1 "KEYSW" H 8150 2900 60  0001 C CNN
-F 2 "ferris:SW_PG1350" H 8150 3000 60  0001 C CNN
+F 2 "ferris:Kailh_PG1232" H 8150 3000 60  0001 C CNN
 F 3 "" H 8150 3000 60  0000 C CNN
 	1    8150 3000
