File: absolem_layout/ferris.kicad_pcb (KiCad board)
At the start: 2 copper layers, 250 x 128.6 mm, 93 parts, among them J1 USB C, K0_0 KEYSW, K0_1 KEYSW, K0_2 KEYSW, K0_3 KEYSW, K0_4 KEYSW, K0_5 KEYSW, K0_6 KEYSW, K0_7 KEYSW, K0_8 KEYSW, K0_9 KEYSW, K1_0 KEYSW, K1_1 KEYSW, K1_2 KEYSW, K1_3 KEYSW, K1_4 KEYSW, K1_5 KEYSW, K1_6 KEYSW, K1_7 KEYSW, K1_8 KEYSW, K1_9 KEYSW, K2_0 KEYSW, K2_1 KEYSW, K2_2 KEYSW, K2_3 KEYSW, K2_4 KEYSW, K2_5 KEYSW, K2_6 KEYSW, K2_7 KEYSW, K2_8 KEYSW, K2_9 KEYSW, K3_2 KEYSW, K3_3 KEYSW, K3_4 KEYSW, K3_5 KEYSW, K3_6 KEYSW, K3_7 KEYSW, SW1 SW_PUSH, U1 ATmega32U4-AU, Y1 Crystal

Commit message: Fixed some staggering
Parts:
- moved K1_7 73.3 mm to (214.9, 48.4)
- moved K2_7 73.3 mm to (221.4, 66.3)
- moved K0_7 73.2 mm to (208.4, 30.5)
- moved K2_8 71.9 mm to (241.7, 66.3)
- moved K1_8 71.7 mm to (235.2, 48.4)
- moved K0_8 71.6 mm to (228.7, 30.5)
- moved C7 70.5 mm to (157.1, 64.4)
- moved J1 70.5 mm to (150.0, 60.8)
- moved C8 70.5 mm to (157.0, 60.3)
- moved C4 70.5 mm to (143.0, 60.3)
- moved R1 70.5 mm to (140.7, 60.4)
- moved SW1 70.5 mm to (140.7, 65.5)
- moved R2 70.5 mm to (159.3, 60.3)
- moved C6 70.5 mm to (159.3, 64.4)
- moved K1_6 69.4 mm to (200.8, 65.2)
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Connections:
- D1 pad 2: (no net) -> Net-(D1-Pad2)
- J1 pad A8: (no net) -> Net-(J1-PadA8)
- J1 pad B8: (no net) -> Net-(J1-PadB8)
- U1 pad 1: (no net) -> Net-(U1-Pad1)
- U1 pad 12: (no net) -> Net-(U1-Pad12)
- U1 pad 18: (no net) -> Net-(U1-Pad18)
- U1 pad 19: (no net) -> Net-(U1-Pad19)
- U1 pad 20: (no net) -> Net-(U1-Pad20)
- U1 pad 21: (no net) -> Net-(U1-Pad21)
- U1 pad 22: (no net) -> Net-(U1-Pad22)
- U1 pad 31: (no net) -> Net-(U1-Pad31)
- U1 pad 32: (no net) -> Net-(U1-Pad32)
- U1 pad 42: (no net) -> Net-(U1-Pad42)
- U1 pad 8: (no net) -> Net-(U1-Pad8)
Routing:
- net /row0,0: track 324.3 -> 174.9 mm, vias 3 -> 2
- net /col0: track 181.4 -> 41.0 mm
- net /row0,1: track 263.9 -> 142.0 mm
- net /col1: track 163.2 -> 44.3 mm
- net /row0,2: track 271.1 -> 154.9 mm
- net /col2: track 158.6 -> 71.3 mm
- net /col3: track 145.2 -> 68.5 mm
- net /col4: track 145.6 -> 87.2 mm
- net Net-(D0_4-Pad2): track 3.56 -> 0.00 mm
- net Net-(D0_1-Pad2): track 3.53 -> 0.00 mm
- net Net-(D0_2-Pad2): track 3.50 -> 0.00 mm
- net Net-(D0_3-Pad2): track 3.49 -> 0.00 mm
- net Net-(D2_2-Pad2): track 3.48 -> 0.00 mm
- net Net-(D0_0-Pad2): track 3.48 -> 0.00 mm
- net Net-(D2_4-Pad2): track 3.33 -> 0.00 mm
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- removed copper zone on B.Cu, net (none)
Other:
- board size 250 x 128.6 mm -> 258.4 x 139.4 mm
- board text added: "Ferris High + Absolem"
- board text added: "by @pierrec83 and Melinda Birkenstock and /u/mrzealot"
- board text removed: "Ferris High v0.1"
- board text removed: "by @pierrec83 and Melinda Birkenstock"

Commit message: Fixed some minor routing and silksscreen
Parts:
- added GFRONT: LOGO, ferris:front, F.Cu at (153.7, 95.9)
- moved R2 49.0 mm to (160.7, 109.2), turned to 90 degrees
- moved D1_0 11.1 mm to (45.4, 48.3)
- moved D1_2 10.8 mm to (92.6, 39.2)
- moved D2_0 10.7 mm to (40.0, 66.7)
- moved D2_2 10.7 mm to (85.9, 57.0)
- moved D0_2 10.5 mm to (99.1, 21.3)
- moved D0_0 10.4 mm to (49.5, 29.6)
- moved D2_7 9.26 mm to (222.8, 56.1)
- moved D1_7 9.12 mm to (215.9, 38.3)
- moved D1_1 9.07 mm to (72.3, 39.2)
- moved D2_1 8.90 mm to (65.5, 57.0)
- moved D0_1 8.68 mm to (78.8, 21.3)
- moved D2_8 8.12 mm to (243.1, 56.1)
- moved D2_3 8.06 mm to (100.3, 73.7)
- moved D0_7 7.24 mm to (207.0, 21.9)
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Connections:
- D1 pad 2: Net-(D1-Pad2) -> (no net)
- J1 pad A8: Net-(J1-PadA8) -> (no net)
- J1 pad B8: Net-(J1-PadB8) -> (no net)
- U1 pad 1: Net-(U1-Pad1) -> (no net)
- U1 pad 12: Net-(U1-Pad12) -> (no net)
- U1 pad 18: Net-(U1-Pad18) -> (no net)
- U1 pad 19: Net-(U1-Pad19) -> (no net)
- U1 pad 20: Net-(U1-Pad20) -> (no net)
- U1 pad 21: Net-(U1-Pad21) -> (no net)
- U1 pad 22: Net-(U1-Pad22) -> (no net)
- U1 pad 25: Net-(D1-Pad4) -> (no net)
- U1 pad 31: Net-(U1-Pad31) -> (no net)
- U1 pad 32: Net-(U1-Pad32) -> Net-(D1-Pad4)
- U1 pad 42: Net-(U1-Pad42) -> (no net)
- U1 pad 8: Net-(U1-Pad8) -> (no net)
Routing:
- net /row0,1: track 142.0 -> 282.0 mm, vias 3 -> 4
- net /col0: track 41.0 -> 174.0 mm
- net /row0,0: track 174.9 -> 307.3 mm, vias 2 -> 3
- net /row0,2: track 154.9 -> 287.2 mm
- net /col1: track 44.3 -> 170.0 mm
- net /col2: track 71.3 -> 157.6 mm
- net /col3: track 68.5 -> 140.2 mm
- net /col4: track 87.2 -> 143.4 mm
- net GND: track 143.6 -> 176.7 mm, vias 7 -> 9
- net Net-(R2-Pad2): track 39.6 -> 8.51 mm
- net Net-(D1-Pad4): track 22.2 -> 6.57 mm, vias 2 -> 0
- net +5V: track 124.2 -> 136.1 mm
- net /col9: track 160.9 -> 150.0 mm, vias 4 -> 2
- net VCC: track 14.0 -> 22.5 mm
- net Net-(J1-PadA7): track 10.1 -> 17.0 mm
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Other:
- board text added: "by @pierrec83, Melinda Birkenstock and /u/mrzealot"
- board text added: "“It's still magic even if you know how it's done.”"
- board text removed: "by @pierrec83 and Melinda Birkenstock and /u/mrzealot"

Commit message: Computer change
Parts:
- added S1: , MX, F.Cu at (30.6, 75.4)
- added S10: , MX, F.Cu at (88.7, 84.2)
- added S11: , MX, F.Cu at (95.2, 66.3)
- added S12: , MX, F.Cu at (101.7, 48.4)
- added S13: , MX, F.Cu at (105.8, 92.5)
- added S14: , MX, F.Cu at (112.3, 74.7)
- added S15: , MX, F.Cu at (118.8, 56.8)
- added S17: , MX, F.Cu at (113.2, 122.4)
- added S19: , MX, F.Cu at (123.9, 142.5)
- added S2: , MX, F.Cu at (35.5, 57.0)
- added S20: , MX, F.Cu at (94.3, 109.7)
- added S21: , MX, F.Cu at (264.2, 75.4)
- added S22: , MX, F.Cu at (259.2, 57.0)
- added S23: , MX, F.Cu at (254.3, 38.7)
- added S24: , MX, F.Cu at (241.4, 70.2)
- added S25: , MX, F.Cu at (234.9, 52.4)
- added S26: , MX, F.Cu at (228.4, 34.5)
- added S27: , MX, F.Cu at (221.9, 72.0)
- added S28: , MX, F.Cu at (215.4, 54.2)
- added S29: , MX, F.Cu at (208.9, 36.3)
- added S3: , MX, F.Cu at (40.4, 38.7)
- added S30: , MX, F.Cu at (206.1, 84.2)
- added S31: , MX, F.Cu at (199.6, 66.3)
- added S32: , MX, F.Cu at (193.1, 48.4)
- added S33: , MX, F.Cu at (188.9, 92.5)
- added S34: , MX, F.Cu at (182.4, 74.7)
- added S35: , MX, F.Cu at (175.9, 56.8)
- added S37: , MX, F.Cu at (181.6, 122.4)
- added S39: , MX, F.Cu at (170.9, 142.5)
- added S4: , MX, F.Cu at (53.3, 70.2)
- added S40: , MX, F.Cu at (200.5, 109.7)
- added S5: , MX, F.Cu at (59.8, 52.4)
- added S6: , MX, F.Cu at (66.3, 34.5)
- added S7: , MX, F.Cu at (72.9, 72.0)
- added S8: , MX, F.Cu at (79.4, 54.2)
- added S9: , MX, F.Cu at (85.9, 36.3)
- moved G*** 81.0 mm to (234.8, 147.0)
- moved K0_2 12.5 mm to (85.9, 36.3)
- moved K1_2 12.4 mm to (79.4, 54.2)
- moved K2_2 12.4 mm to (72.9, 72.0)
- moved D0_1 11.1 mm to (69.1, 26.8)
- moved D1_1 11.1 mm to (62.6, 44.6)
- moved D2_1 10.9 mm to (56.1, 62.5)
- moved K0_1 10.8 mm to (66.3, 34.5)
- moved K1_1 10.8 mm to (59.8, 52.4)
- moved K2_1 10.8 mm to (53.3, 70.2)
- moved K0_3 8.86 mm to (101.7, 48.4)
- moved K1_3 8.83 mm to (95.2, 66.3)
- moved K2_3 8.80 mm to (88.7, 84.2)
- moved K0_7 8.40 mm to (208.9, 36.3)
- moved K1_7 8.36 mm to (215.4, 54.2)
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Other:
- board text added: "Credits & Rights go to @pierrec83, Melinda Birkenstock (Ferris MX) and MrZealot (Absolem)"
- board text removed: "Ferris High + Absolem"
- board text removed: "by @pierrec83, Melinda Birkenstock and /u/mrzealot"

Commit message: Devid commit
Parts:
- G***: moved to F.Cu
- moved G*** 90.0 mm to (148.0, 123.2), turned to 10 degrees
- moved GFRONT 1.53 mm to (148.2, 95.4)
Routing:
- net /col4: track 143.4 -> 146.8 mm
- net /col3: track 140.2 -> 138.6 mm

Commit message: Connected up most of the power. PCB incomplete still
Parts:
- removed the R2 at (154.8, 110.2)
- removed R3, R4: 22, Resistor_SMD:R_0805_2012Metric_Pad1.15x1.40mm_HandSolder
- removed S1, S10, S11, S12, S13, S14, S15, S17, S19, S2, S20, S21, S22, S23, S24, S25, S26, S27, S28, S29, S3, S30, S31, S32, S33, S34, S35, S37, S39, S4, S40, S5, S6, S7, S8, S9: , MX
- added C10: 30p, Capacitor_SMD:C_0805_2012Metric_Pad1.15x1.40mm_HandSolder, F.Cu at (143.9, 140.3)
- added C11: 100n, Capacitor_SMD:C_0805_2012Metric_Pad1.15x1.40mm_HandSolder, F.Cu at (158.4, 167.4)
- added C9: 100n, Capacitor_SMD:C_0805_2012Metric_Pad1.15x1.40mm_HandSolder, F.Cu at (154.9, 126.0)
- added IC1: NUF2221W1T2G, digikey-footprints:SOT-363, F.Cu at (148.2, 68.6)
- added J2: Conn_01x05_Male, Connector_PinHeader_2.54mm:PinHeader_1x05_P2.54mm_Vertical, F.Cu at (198.8, 147.0)
- added U2: STM32F303CBTx, Package_QFP:LQFP-48_7x7mm_P0.5mm, F.Cu at (147.7, 130.8)
- C1, C2: value 22p -> 1u
- C3: value 0.1u -> 1u
- C4: value 0.1u -> 10n
- C5: value 0.1u -> 4.7u
- C6: value 0.1u -> 30p
- C7: value 4.7u -> 100n
- C8: value 1u -> 100n
- R1: value 10k -> 5.1K
- R5: value 5.1K -> 10k
- U1: value ATmega32U4-AU -> TLV70012_SOT23-5; footprint Package_QFP:TQFP-44_10x10mm_P0.8mm -> Package_TO_SOT_SMD:SOT-23-5
- Y1: value Crystal -> 8MHz; footprint Crystal:Crystal_SMD_3225-4Pin_3.2x2.5mm -> Crystal:Crystal_SMD_5032-4Pin_5.0x3.2mm
- moved C8 106.5 mm to (216.7, 146.2), turned to 0 degrees
- moved C4 77.8 mm to (152.7, 136.3)
- moved C6 77.1 mm to (152.0, 140.3)
- moved C7 61.4 mm to (143.3, 123.7), turned to 270 degrees
- moved R5 57.6 mm to (140.5, 132.7)
- moved D1 52.4 mm to (133.7, 59.6), turned to 180 degrees
- moved Y1 45.1 mm to (148.0, 140.3), turned to 180 degrees
- moved C3 37.7 mm to (154.8, 136.3), turned to 90 degrees
- moved C1 36.0 mm to (134.5, 64.5), turned to 90 degrees
- moved C5 34.4 mm to (141.4, 123.7), turned to 270 degrees
- moved U1 32.6 mm to (138.4, 65.0)
- moved G*** 31.6 mm to (146.1, 91.7)
- moved C2 25.6 mm to (141.5, 67.4), turned to 90 degrees
- moved SW1 19.7 mm to (157.9, 59.4)
- moved R2 19.0 mm to (141.2, 58.9), turned to 270 degrees
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- renumbered D0_0 to D0_1, D0_9 to D0_10, D0_1 to D0_2, D0_2 to D0_3, D0_3 to D0_4, D0_4 to D0_5, D0_5 to D0_6, D0_6 to D0_7, D0_7 to D0_8, D0_8 to D0_9, D1_0 to D1_1, D1_9 to D1_10, D1_1 to D1_2, D1_2 to D1_3, D1_3 to D1_4, D1_4 to D1_5, D1_5 to D1_6, D1_6 to D1_7, D1_7 to D1_8, D1_8 to D1_9, D2_0 to D2_1, D2_9 to D2_10, D2_1 to D2_2, D2_2 to D2_3, D2_3 to D2_4, D2_4 to D2_5, D2_5 to D2_6, D2_6 to D2_7, D2_7 to D2_8, D2_8 to D2_9, D3_2 to D3_1, D3_3 to D3_2, D3_4 to D3_3, D3_5 to D3_4, D3_6 to D3_5, D3_7 to D3_6, K0_0 to K0_1, K0_9 to K0_10, K0_1 to K0_2, K0_2 to K0_3, K0_3 to K0_4, K0_4 to K0_5, K0_5 to K0_6, K0_6 to K0_7, K0_7 to K0_8, K0_8 to K0_9, K1_0 to K1_1, K1_9 to K1_10, K1_1 to K1_2, K1_2 to K1_3, K1_3 to K1_4, K1_4 to K1_5, K1_5 to K1_6, K1_6 to K1_7, K1_7 to K1_8, K1_8 to K1_9, K2_0 to K2_1, K2_9 to K2_10, K2_1 to K2_2, K2_2 to K2_3, K2_3 to K2_4, K2_4 to K2_5, K2_5 to K2_6, K2_6 to K2_7, K2_7 to K2_8, K2_8 to K2_9, K3_2 to K3_1, K3_3 to K3_2, K3_4 to K3_3, K3_5 to K3_4, K3_6 to K3_5, K3_7 to K3_6, R6 to R2
Connections:
- net Net-(J1-PadA6) renamed /D+I
- net Net-(J1-PadA7) renamed /D-I
- net VCC renamed Net-(F1-Pad2)
- C1 pad 1: Net-(C1-Pad1) -> GND
- C1 pad 2: GND -> +5V
- C2 pad 1: GND -> +3V3
- C2 pad 2: Net-(C2-Pad2) -> GND
- C3 pad 1: +5V -> GND
- C3 pad 2: GND -> +3V3
- C4 pad 1: +5V -> GND
- C4 pad 2: GND -> +3V3
- C5 pad 1: +5V -> GND
- C5 pad 2: GND -> +3V3
- C6 pad 1: +5V -> GND
- C6 pad 2: GND -> /OSC_OUT
- C7 pad 1: +5V -> GND
- C7 pad 2: GND -> +3V3
- C8 pad 1: Net-(C8-Pad1) -> GND
- C8 pad 2: GND -> +3V3
- D0_1 pad 1: /row0,0 -> /row0
- D0_10 pad 1: /row0,0 -> /row0
- D0_2 pad 1: /row0,0 -> /row0
- D0_3 pad 1: /row0,0 -> /row0
- D0_4 pad 1: /row0,0 -> /row0
- D0_5 pad 1: /row0,0 -> /row0
- D0_6 pad 1: /row0,0 -> /row0
- D0_7 pad 1: /row0,0 -> /row0
- D0_8 pad 1: /row0,0 -> /row0
- D0_9 pad 1: /row0,0 -> /row0
- D1 pad 4: Net-(D1-Pad4) -> /LAYER_LED
- D1_1 pad 1: /row0,1 -> /row1
- D1_10 pad 1: /row0,1 -> /row1
- D1_2 pad 1: /row0,1 -> /row1
- D1_3 pad 1: /row0,1 -> /row1
- D1_4 pad 1: /row0,1 -> /row1
- D1_5 pad 1: /row0,1 -> /row1
- D1_6 pad 1: /row0,1 -> /row1
- D1_7 pad 1: /row0,1 -> /row1
- D1_8 pad 1: /row0,1 -> /row1
- D1_9 pad 1: /row0,1 -> /row1
- D2_1 pad 1: /row0,2 -> /row2
- D2_10 pad 1: /row0,2 -> /row2
- D2_2 pad 1: /row0,2 -> /row2
- D2_3 pad 1: /row0,2 -> /row2
- D2_4 pad 1: /row0,2 -> /row2
- D2_5 pad 1: /row0,2 -> /row2
- D2_6 pad 1: /row0,2 -> /row2
- D2_7 pad 1: /row0,2 -> /row2
- D2_8 pad 1: /row0,2 -> /row2
- D2_9 pad 1: /row0,2 -> /row2
- D3_1 pad 1: /row0,3 -> /row3
- D3_2 pad 1: /row0,3 -> /row3
- D3_3 pad 1: /row0,3 -> /row3
- D3_4 pad 1: /row0,3 -> /row3
- D3_5 pad 1: /row0,3 -> /row3
- D3_6 pad 1: /row0,3 -> /row3
- R1 pad 1: Net-(R1-Pad1) -> GND
- R1 pad 2: +5V -> Net-(J1-PadA5)
- R5 pad 2: Net-(J1-PadA5) -> Net-(R5-Pad2)
- SW1 pad 1: GND -> +3V3
- SW1 pad 2: Net-(R1-Pad1) -> Net-(R5-Pad2)
- U1 pad 1: (no net) -> +5V
- U1 pad 2: +5V -> GND
- U1 pad 3: /D- -> +5V
- U1 pad 4: /D+ -> (no net)
- U1 pad 5: GND -> +3V3
- Y1 pad 1: Net-(C1-Pad1) -> /OSC_OUT
- Y1 pad 3: Net-(C2-Pad2) -> /OSC_IN
Routing:
- net /row0,0: track 307.3 -> 0.00 mm, vias 3 -> 0
- net /row0,2: track 287.2 -> 0.00 mm, vias 4 -> 0
- net /row0,1: track 282.0 -> 0.00 mm, vias 4 -> 0
- net /row0: track 0.00 -> 232.3 mm, vias 0 -> 4
- net /row0,3: track 194.1 -> 0.00 mm, vias 6 -> 0
- net /col0: track 174.0 -> 0.00 mm
- net /col1: track 170.0 -> 0.00 mm, vias 2 -> 0
- net /row2: track 0.00 -> 161.8 mm
- net /col2: track 157.6 -> 0.95 mm, vias 1 -> 0
- net /row3: track 0.00 -> 155.9 mm, vias 0 -> 4
- net +3V3: track 0.00 -> 144.1 mm, vias 0 -> 6
- net /col8: track 142.4 -> 0.00 mm, vias 4 -> 0
- net /col6: track 139.2 -> 0.00 mm, vias 2 -> 0
- net /col3: track 138.6 -> 0.97 mm
- net +5V: track 136.1 -> 16.9 mm, vias 5 -> 0
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Other:
- net class Power: trace_width 0.381 -> 0.254

Commit message: Updated the routing and positons
Parts:
- removed C11, C8: 100n, Capacitor_SMD:C_0805_2012Metric_Pad1.15x1.40mm_HandSolder
- removed J2: Conn_01x05_Male, Connector_PinHeader_2.54mm:PinHeader_1x05_P2.54mm_Vertical
- moved D0_8 12.4 mm to (208.9, 32.5)
- moved D1_8 12.4 mm to (215.4, 50.4)
- moved D2_8 12.3 mm to (221.9, 68.3)
- moved D0_3 10.6 mm to (91.7, 32.7)
- moved D2_3 10.5 mm to (78.8, 68.4)
- moved D1_3 10.5 mm to (85.2, 50.6)
- moved D2_9 10.2 mm to (241.1, 66.5)
- moved D0_9 9.74 mm to (228.1, 30.8)
- moved D1_9 9.64 mm to (234.6, 48.7)
- moved D0_7 6.92 mm to (192.9, 44.7)
- moved D1_7 6.87 mm to (199.4, 62.6)
- moved D2_7 6.86 mm to (205.9, 80.4)
- moved D0_4 5.86 mm to (107.4, 44.8)
- moved D1_4 5.81 mm to (100.9, 62.6)
- moved D2_4 5.76 mm to (94.4, 80.5)
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Connections:
- U2 pad 14: /row2 -> /col5
- U2 pad 15: /row1 -> /col6
- U2 pad 16: /row0 -> /col7
- U2 pad 26: /col6 -> (no net)
- U2 pad 27: /col3 -> /col9
- U2 pad 28: /col2 -> /col8
- U2 pad 29: /col1 -> /row2
- U2 pad 30: /col0 -> /row1
- U2 pad 31: /col5 -> /row0
- U2 pad 40: /col9 -> /col1
- U2 pad 41: /col8 -> /col0
- U2 pad 42: /col7 -> /col2
- U2 pad 43: (no net) -> /col3
Routing:
- net /row1: track 0.00 -> 321.8 mm, vias 0 -> 6
- net /col0: track 0.00 -> 171.7 mm
- net /row2: track 161.8 -> 330.8 mm, vias 0 -> 6
- net /col1: track 0.00 -> 157.6 mm
- net /col8: track 0.00 -> 154.2 mm
- net /col2: track 0.95 -> 148.0 mm
- net /col9: track 38.1 -> 163.7 mm
- net /col3: track 0.97 -> 126.4 mm
- net /col6: track 0.00 -> 122.4 mm
- net /row0: track 232.3 -> 332.8 mm, vias 4 -> 6
- net /col7: track 54.2 -> 145.3 mm, vias 0 -> 3
- net /col4: track 82.0 -> 119.4 mm
- net Net-(R5-Pad2): track 116.6 -> 91.7 mm
- net /col5: track 99.9 -> 122.0 mm, vias 0 -> 1
- net /row3: track 155.9 -> 173.2 mm, vias 4 -> 8
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